Commit message: Added mesh files to urdf

File: src/robot_urdf/urdf/robot.urdf.xacro (robot description, xacro)
@@ -27,14 +27,13 @@
     <visual>
       <geometry>
+        <mesh filename="package://robot_urdf/meshes/base.stl"/>
+      </geometry>
+      <origin rpy="1.57075 0 1.57075" xyz="-0.08 -0.525 0.0"/>
+    </visual>
+    <collision>
+      <geometry>
         <box size="${baseLength} ${baseWidth} ${baseHeight}"/>
       </geometry>
-      <material name="blue"/>
-      <origin rpy="0 0 0" xyz="0 0 0.3"/>
-    </visual>
-    <collision>
-      <geometry>
-        <box size="${baseLength} ${baseWidth} ${baseHeight}"/>
-      </geometry>
-      <origin rpy="0 0 0" xyz="0 0 0.3"/>
+      <origin rpy="0 0 0" xyz="0 0 0.0"/>
     </collision>
     <inertial>

Commit message: Added urdf features

File: src/robot_urdf/urdf/robot.urdf.xacro (robot description, xacro)
@@ -2,17 +2,17 @@
 <robot xmlns:xacro="http://www.ros.org/wiki/xacro" name="robot">
   <material name="blue">
-    <color rgba="0 0 0.8 .5"/>
+    <color rgba="0 0 0.8 1.0"/>
   </material>
   <material name="black">
-    <color rgba="0 0 0 0.5"/>
+    <color rgba="0.3 0.3 0.3 0.9"/>
   </material>
   <material name="white">
-    <color rgba="1 1 1 .5"/>
+    <color rgba="1 1 1 0.6"/>
   </material>
   <material name="green">
-    <color rgba="0 1 0 0.5"/>
+    <color rgba="0 1 0"/>
   </material>
   <xacro:property name="baseLength" value="1.029" />
-  <xacro:property name="baseWidth" value="0.838" />
+  <xacro:property name="baseWidth" value="0.58" />
   <xacro:property name="baseHeight" value="0.686" />
   <xacro:property name="baseMass" value="27" />
@@ -24,4 +24,5 @@
   <xacro:property name="camWidth" value="0.1016" />
   <xacro:property name="camRadius" value="0.0127" />
+<!-- Base -->
   <link name="base_link">
     <visual>
@@ -30,10 +31,17 @@
       </geometry>
       <origin rpy="1.57075 0 1.57075" xyz="-0.08 -0.525 0.0"/>
-    </visual>
-    <collision>
-      <geometry>
-        <box size="${baseLength} ${baseWidth} ${baseHeight}"/>
-      </geometry>
-      <origin rpy="0 0 0" xyz="0 0 0.0"/>
+      <material name="blue"/>
+    </visual>
+    <collision>
+      <geometry>
+        <box size="0.68 0.68 0.36"/>
+      </geometry>
+      <origin rpy="0 0 0" xyz="0.1 0 0.221"/>
+    </collision>
+    <collision>
+      <geometry>
+        <box size="0.3 0.68 0.15"/>
+      </geometry>
+      <origin rpy="0 0 0" xyz="-0.32 0 0.08"/>
     </collision>
     <inertial>
@@ -42,103 +50,205 @@
     </inertial>
   </link>
+<!-- Right Wheels -->
   <link name="front_right_wheel">
     <visual>
       <geometry>
-        <cylinder length="${wheelWidth}" radius="${wheelRadius}"/>
-      </geometry>
-      <origin rpy="0 1.57075 1.57075" xyz="0 ${-wheelWidth/2} 0"/>
-      <material name="white"/>
-    </visual>
-    <collision>
-      <geometry>
-        <cylinder length="${wheelWidth}" radius="${wheelRadius}"/>
-      </geometry>
-      <origin rpy="0 1.57075 1.57075" xyz="0 ${-wheelWidth/2} 0"/>
-    </collision>
-    <inertial>
-      <mass value="${wheelMass}"/>
-      <inertia ixx="0.4" ixy="0.0" ixz="0.0" iyy="0.4" iyz="0.0" izz="0.2"/>
-    </inertial>
-  </link>
-  <joint name="base_to_front_right_wheel" type="continuous">
+        <mesh filename="package://robot_urdf/meshes/wheel.stl"/>
+      </geometry>
+      <origin rpy="0 1.57075 1.57075" xyz="0 ${-wheelWidth/2} 0"/>
+      <material name="black"/>
+    </visual>
+    <collision>
+      <geometry>
+        <cylinder length="${wheelWidth}" radius="${wheelRadius}"/>
+      </geometry>
+      <origin rpy="0 1.57075 1.57075" xyz="0 ${-wheelWidth/2} 0"/>
+    </collision>
+    <inertial>
+      <mass value="${wheelMass}"/>
+      <inertia ixx="0.4" ixy="0.0" ixz="0.0" iyy="0.4" iyz="0.0" izz="0.2"/>
+    </inertial>
+  </link>
+  <joint name="base_to_front_right_wheel" type="fixed">
     <parent link="base_link"/>
     <child link="front_right_wheel"/>
     <axis xyz="0 1 0"/>
-    <origin xyz="${wheelOffset} ${-baseWidth /2} 0"/>
+    <origin xyz="0.315 ${-baseWidth /2} 0.028"/>
+  </joint>
+  <link name="front_middle_right_wheel">
+    <visual>
+      <geometry>
+        <mesh filename="package://robot_urdf/meshes/wheel.stl"/>
+      </geometry>
+      <origin rpy="0 1.57075 1.57075" xyz="0 ${-wheelWidth/2} 0"/>
+      <material name="black"/>
+    </visual>
+    <collision>
+      <geometry>
+        <cylinder length="${wheelWidth}" radius="${wheelRadius}"/>
+      </geometry>
+      <origin rpy="0 1.57075 1.57075" xyz="0 ${-wheelWidth/2} 0"/>
+    </collision>
+    <inertial>
+      <mass value="${wheelMass}"/>
+      <inertia ixx="0.4" ixy="0.0" ixz="0.0" iyy="0.4" iyz="0.0" izz="0.2"/>
+    </inertial>
+  </link>
+  <joint name="base_to_front_middle_right_wheel" type="fixed">
+    <parent link="base_link"/>
+    <child link="front_middle_right_wheel"/>
+    <axis xyz="0 1 0"/>
+    <origin xyz="0.104 ${-baseWidth /2} 0.022"/>
+  </joint>
+  <link name="back_middle_right_wheel">
+    <visual>
+      <geometry>
+        <mesh filename="package://robot_urdf/meshes/wheel.stl"/>
+      </geometry>
+      <origin rpy="0 1.57075 1.57075" xyz="0 ${-wheelWidth/2} 0"/>
+      <material name="black"/>
+    </visual>
+    <collision>
+      <geometry>
+        <cylinder length="${wheelWidth}" radius="${wheelRadius}"/>
+      </geometry>
+      <origin rpy="0 1.57075 1.57075" xyz="0 ${-wheelWidth/2} 0"/>
+    </collision>
+    <inertial>
+      <mass value="${wheelMass}"/>
+      <inertia ixx="0.4" ixy="0.0" ixz="0.0" iyy="0.4" iyz="0.0" izz="0.2"/>
+    </inertial>
+  </link>
+  <joint name="base_to_back_middle_right_wheel" type="fixed">
+    <parent link="base_link"/>
+    <child link="back_middle_right_wheel"/>
+    <axis xyz="0 1 0"/>
+    <origin xyz="-0.122 ${-baseWidth /2} 0.022"/>
   </joint>
   <link name="back_right_wheel">
     <visual>
       <geometry>
-        <cylinder length="${wheelWidth}" radius="${wheelRadius}"/>
-      </geometry>
-      <origin rpy="0 1.57075 1.57075" xyz="0 ${-wheelWidth/2} 0"/>
-      <material name="white"/>
-    </visual>
-    <collision>
-      <geometry>
-        <cylinder length="${wheelWidth}" radius="${wheelRadius}"/>
-      </geometry>
-      <origin rpy="0 1.57075 1.57075" xyz="0 ${-wheelWidth/2} 0"/>
-    </collision>
-    <inertial>
-      <mass value="${wheelMass}"/>
-      <inertia ixx="0.4" ixy="0.0" ixz="0.0" iyy="0.4" iyz="0.0" izz="0.2"/>
-    </inertial>
-  </link>
-  <joint name="base_to_back_right_wheel" type="continuous">
+        <mesh filename="package://robot_urdf/meshes/wheel.stl"/>
+      </geometry>
+      <origin rpy="0 1.57075 1.57075" xyz="0 ${-wheelWidth/2} 0"/>
+      <material name="black"/>
+    </visual>
+    <collision>
+      <geometry>
+        <cylinder length="${wheelWidth}" radius="${wheelRadius}"/>
+      </geometry>
+      <origin rpy="0 1.57075 1.57075" xyz="0 ${-wheelWidth/2} 0"/>
+    </collision>
+    <inertial>
+      <mass value="${wheelMass}"/>
+      <inertia ixx="0.4" ixy="0.0" ixz="0.0" iyy="0.4" iyz="0.0" izz="0.2"/>
+    </inertial>
+  </link>
+  <joint name="base_to_back_right_wheel" type="fixed">
     <parent link="base_link"/>
     <child link="back_right_wheel"/>
     <axis xyz="0 1 0"/>
-    <origin xyz="${-wheelOffset} ${-baseWidth /2} 0"/>
-  </joint>
+    <origin xyz="-0.334 ${-baseWidth /2} 0.028"/>
+  </joint>
+<!-- Left Wheels -->
   <link name="front_left_wheel">
     <visual>
       <geometry>
-        <cylinder length="${wheelWidth}" radius="${wheelRadius}"/>
-      </geometry>
-      <origin rpy="0 1.57075 1.57075" xyz="0 ${wheelWidth/2} 0"/>
-      <material name="white"/>
-    </visual>
-    <collision>
-      <geometry>
-        <cylinder length="${wheelWidth}" radius="${wheelRadius}"/>
-      </geometry>
-      <origin rpy="0 1.57075 1.57075" xyz="0 ${wheelWidth/2} 0"/>
-    </collision>
-    <inertial>
-      <mass value="${wheelMass}"/>
-      <inertia ixx="0.4" ixy="0.0" ixz="0.0" iyy="0.4" iyz="0.0" izz="0.2"/>
-    </inertial>
-  </link>
-  <joint name="base_to_front_left_wheel" type="continuous">
+        <mesh filename="package://robot_urdf/meshes/wheel.stl"/>
+      </geometry>
+      <origin rpy="0 1.57075 1.57075" xyz="0 ${wheelWidth/2} 0"/>
+      <material name="black"/>
+    </visual>
+    <collision>
+      <geometry>
+        <cylinder length="${wheelWidth}" radius="${wheelRadius}"/>
+      </geometry>
+      <origin rpy="0 1.57075 1.57075" xyz="0 ${wheelWidth/2} 0"/>
+    </collision>
+    <inertial>
+      <mass value="${wheelMass}"/>
+      <inertia ixx="0.4" ixy="0.0" ixz="0.0" iyy="0.4" iyz="0.0" izz="0.2"/>
+    </inertial>
+  </link>
+  <joint name="base_to_front_left_wheel" type="fixed">
     <parent link="base_link"/>
     <child link="front_left_wheel"/>
     <axis xyz="0 1 0"/>
-    <origin xyz="${wheelOffset} ${baseWidth /2} 0"/>
+    <origin xyz="0.315 ${baseWidth /2} 0.028"/>
+  </joint>
+  <link name="front_middle_left_wheel">
+    <visual>
+      <geometry>
+        <mesh filename="package://robot_urdf/meshes/wheel.stl"/>
+      </geometry>
+      <origin rpy="0 1.57075 1.57075" xyz="0 ${wheelWidth/2} 0"/>
+      <material name="black"/>
+    </visual>
+    <collision>
+      <geometry>
+        <cylinder length="${wheelWidth}" radius="${wheelRadius}"/>
+      </geometry>
+      <origin rpy="0 1.57075 1.57075" xyz="0 ${wheelWidth/2} 0"/>
+    </collision>
+    <inertial>
+      <mass value="${wheelMass}"/>
+      <inertia ixx="0.4" ixy="0.0" ixz="0.0" iyy="0.4" iyz="0.0" izz="0.2"/>
+    </inertial>
+  </link>
+  <joint name="base_to_front_middle_left_wheel" type="fixed">
+    <parent link="base_link"/>
+    <child link="front_middle_left_wheel"/>
+    <axis xyz="0 1 0"/>
+    <origin xyz="0.104 ${baseWidth /2} 0.022"/>
+  </joint>
+  <link name="back_middle_left_wheel">
+    <visual>
+      <geometry>
+        <mesh filename="package://robot_urdf/meshes/wheel.stl"/>
+      </geometry>
+      <origin rpy="0 1.57075 1.57075" xyz="0 ${wheelWidth/2} 0"/>
+      <material name="black"/>
+    </visual>
+    <collision>
+      <geometry>
+        <cylinder length="${wheelWidth}" radius="${wheelRadius}"/>
+      </geometry>
+      <origin rpy="0 1.57075 1.57075" xyz="0 ${wheelWidth/2} 0"/>
+    </collision>
+    <inertial>
+      <mass value="${wheelMass}"/>
+      <inertia ixx="0.4" ixy="0.0" ixz="0.0" iyy="0.4" iyz="0.0" izz="0.2"/>
+    </inertial>
+  </link>
+  <joint name="base_to_back_middle_left_wheel" type="fixed">
+    <parent link="base_link"/>
+    <child link="back_middle_left_wheel"/>
+    <axis xyz="0 1 0"/>
+    <origin xyz="-0.122 ${baseWidth /2} 0.022"/>
   </joint>
   <link name="back_left_wheel">
     <visual>
       <geometry>
-        <cylinder length="${wheelWidth}" radius="${wheelRadius}"/>
-      </geometry>
-      <origin rpy="0 1.57075 1.57075" xyz="0 ${wheelWidth/2} 0"/>
-      <material name="white"/>
-    </visual>
-    <collision>
-      <geometry>
-        <cylinder length="${wheelWidth}" radius="${wheelRadius}"/>
-      </geometry>
-      <origin rpy="0 1.57075 1.57075" xyz="0 ${-wheelWidth/2} 0"/>
-    </collision>
-    <inertial>
-      <mass value="${wheelMass}"/>
-      <inertia ixx="0.4" ixy="0.0" ixz="0.0" iyy="0.4" iyz="0.0" izz="0.2"/>
-    </inertial>
-  </link>
-  <joint name="base_to_back_left_wheel" type="continuous">
+        <mesh filename="package://robot_urdf/meshes/wheel.stl"/>
+      </geometry>
+      <origin rpy="0 1.57075 1.57075" xyz="0 ${wheelWidth/2} 0"/>
+      <material name="black"/>
+    </visual>
+    <collision>
+      <geometry>
+        <cylinder length="${wheelWidth}" radius="${wheelRadius}"/>
+      </geometry>
+      <origin rpy="0 1.57075 1.57075" xyz="0 ${wheelWidth/2} 0"/>
+    </collision>
+    <inertial>
+      <mass value="${wheelMass}"/>
+      <inertia ixx="0.4" ixy="0.0" ixz="0.0" iyy="0.4" iyz="0.0" izz="0.2"/>
+    </inertial>
+  </link>
+  <joint name="base_to_back_left_wheel" type="fixed">
     <parent link="base_link"/>
     <child link="back_left_wheel"/>
     <axis xyz="0 1 0"/>
-    <origin xyz="${-wheelOffset} ${baseWidth /2} 0"/>
+    <origin xyz="-0.334 ${baseWidth /2} 0.028"/>
   </joint>
   <!-- Intake -->
@@ -146,25 +256,31 @@
     <visual>
       <geometry>
-        <cylinder length="${wheelWidth}" radius="${wheelRadius}"/>
-      </geometry>
-      <origin rpy="0 0 0" xyz="0 0 0"/>
+        <mesh filename="package://robot_urdf/meshes/intake.stl"/>
+      </geometry>
+      <origin rpy="3.14159265 0 0" xyz="-0.272 0.506 0.288"/>
       <material name="white"/>
     </visual>
     <collision>
       <geometry>
-        <cylinder length="${wheelWidth}" radius="${wheelRadius}"/>
-      </geometry>
-      <origin rpy="0 0 0" xyz="0 0 0"/>
-    </collision>
-    <inertial>
-      <mass value="${wheelMass}"/>
-      <inertia ixx="0.4" ixy="0.0" ixz="0.0" iyy="0.4" iyz="0.0" izz="0.2"/>
-    </inertial>
-  </link>
-  <joint name="intake_to_base_link" type="fixed">
+        <box size="0.36 0.63 0.09"/>
+      </geometry>
+      <origin rpy="0 0 0" xyz="-0.17 0 0.015"/>
+    </collision>
+    <collision>
+      <geometry>
+        <box size="0.1 0.63 0.13"/>
+      </geometry>
+      <origin rpy="0 0 0" xyz="-0.3 0 -0.03"/>
+    </collision>
+    <inertial>
+      <mass value="${wheelMass}"/>
+      <inertia ixx="0.4" ixy="0.0" ixz="0.0" iyy="0.4" iyz="0.0" izz="0.2"/>
+    </inertial>
+  </link>
+  <joint name="intake_to_base_link" type="continuous">
     <parent link="base_link"/>
     <child link="intake_link"/>
     <axis xyz="0 1 0"/>
-    <origin xyz="${-wheelOffset-0.3} 0 0"/>
+    <origin xyz="-0.296 0 0.2"/>
   </joint>
   <!-- Turret -->
@@ -172,25 +288,25 @@
     <visual>
       <geometry>
-        <cylinder length="${wheelWidth}" radius="${wheelRadius}"/>
-      </geometry>
-      <origin rpy="0 0 0" xyz="0 0 0"/>
+        <mesh filename="package://robot_urdf/meshes/turret.stl"/>
+      </geometry>
+      <origin rpy="1.57075 0 0" xyz="-0.12 0.23 -0.12"/>
       <material name="white"/>
     </visual>
     <collision>
       <geometry>
-        <cylinder length="${wheelWidth}" radius="${wheelRadius}"/>
-      </geometry>
-      <origin rpy="0 0 0" xyz="0 0 0"/>
-    </collision>
-    <inertial>
-      <mass value="${wheelMass}"/>
-      <inertia ixx="0.4" ixy="0.0" ixz="0.0" iyy="0.4" iyz="0.0" izz="0.2"/>
-    </inertial>
-  </link>
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
Commit message: added joy stick control

File: src/robot_urdf/urdf/robot.urdf.xacro (robot description, xacro)
@@ -41,7 +41,7 @@
     <collision>
       <geometry>
-        <box size="0.3 0.68 0.15"/>
-      </geometry>
-      <origin rpy="0 0 0" xyz="-0.32 0 0.08"/>
+        <box size="0.3 0.68 0.12"/>
+      </geometry>
+      <origin rpy="0 0 0" xyz="-0.32 0 0.1"/>
     </collision>
     <inertial>

Commit message: Added hood to urdf

File: src/robot_urdf/urdf/robot.urdf.xacro (robot description, xacro)
@@ -290,5 +290,5 @@
         <mesh filename="package://robot_urdf/meshes/turret.stl"/>
       </geometry>
-      <origin rpy="1.57075 0 0" xyz="-0.12 0.23 -0.12"/>
+      <origin rpy="1.57075 0 -1.57075" xyz="0.23 0.12 -0.12"/>
       <material name="white"/>
     </visual>
@@ -308,5 +308,50 @@
     <child link="turret_link"/>
     <axis xyz="0 0 1"/>
-    <origin xyz="0.232 0 0.38"/>
+    <origin rpy="0 0 1.57075" xyz="0.232 0 0.38"/>
+  </joint>
+<!-- Hood -->
+  <link name="hood_link">
+    <visual>
+      <geometry>
+        <mesh filename="package://robot_urdf/meshes/hood.stl"/>
+      </geometry>
+      <origin xyz="0.222 0.12 -0.143" rpy="2.059442 0 -1.57075"/>
+      <material name="white"/>
+    </visual>
+    <inertial>
+      <mass value="${wheelMass}"/>
+      <inertia ixx="0.4" ixy="0.0" ixz="0.0" iyy="0.4" iyz="0.0" izz="0.2"/>
+    </inertial>
+  </link>
+  <joint name="hood_to_turret" type="continuous">
+    <parent link="turret_link"/>
+    <child link="hood_link"/>
+    <axis xyz="0 1 0"/>
+    <origin rpy="0 0.488692 0" xyz="0.1 0 0.11"/>
+  </joint>
+  <link name="shoot_angle_link">
+    <inertial>
+      <mass value="${wheelMass}"/>
+      <inertia ixx="0.4" ixy="0.0" ixz="0.0" iyy="0.4" iyz="0.0" izz="0.2"/>
+    </inertial>
+  </link>
+  <joint name="shoot_angle_to_hood" type="fixed">
+    <parent link="hood_link"/>
+    <child link="shoot_angle_link"/>
+    <axis xyz="0 1 0"/>
+    <origin rpy="0 -1.57075 0" xyz="-0.23 0 0.03"/>
+  </joint>
+<!-- Flywheel -->
+  <link name="flywheel_link">
+    <inertial>
+      <mass value="${wheelMass}"/>
+      <inertia ixx="0.4" ixy="0.0" ixz="0.0" iyy="0.4" iyz="0.0" izz="0.2"/>
+    </inertial>
+  </link>
+  <joint name="flywheel_to_turret" type="fixed">
+    <parent link="turret_link"/>
+    <child link="flywheel_link"/>
+    <axis xyz="0 1 0"/>
+    <origin rpy="0 0.0 0" xyz="0.05 0 0.11"/>
   </joint>
   <!-- Sensors -->
@@ -359,5 +404,5 @@
     <child link="d435_link"/>
     <axis xyz="0 1 0"/>
-    <origin rpy="0 -0.523599 1.57075" xyz="0.0 0.2 0.15"/>
+    <origin rpy="0 -0.523599 0" xyz="0.2 0.0 0.15"/>
   </joint>
 </robot>
